File: schematics/Selenium/devBoard.sch (EAGLE design)
At the start: 21 parts, among them J2 629105136821, U1 TSL2591, U5 MCP73831SOT23-5

Commit message: Add enable pin pads for regulator, tidy, then untrack backup files
Parts:
- added R3: 100K, Resistor:R_CHIP-0603(1608-METRIC)
- added TP2, VREG_EN: TESTPOINT_TPS-PAD-036, 52101-101-REV-A_v16:TESTPOINT_TPS-PAD-036
- D1, D2: value (none) -> MBR120
Connections:
- new net N$13: R3.1, VREG_EN.TP
- new net N$14: TP2.TP, U4.EN
- net N$1: now also R3.2
Other:
- moved on the sheet: +3V3, BAT+, BAT-, C1, C4, C5, D2, GND, U4
